Commit message: make visualize an argument

File: mirte_description/mirte_master_description/urdf/mirte_master.xacro (robot description, xacro)
@@ -10,4 +10,5 @@
   <xacro:arg name="depth_camera_enable" default="True" />
   <xacro:arg name="imu_enable" default="True" />
+  <xacro:arg name="visualize_sensors" value="True" />
   <xacro:property name="camera_name" value="camera" lazy_eval="False"/>
   <xacro:property name="namespace" value="" scope="global" lazy_eval="False"/>
@@ -20,5 +21,4 @@
   <xacro:property name="wheel_effort" value="5" />
   <xacro:property name="base_mass" value="5.0" />
-  <xacro:property name="visualize_sensors" value="True" />
   <material name="blue">
     <color rgba="0.203125 0.23828125 0.28515625 1.0" />
