Commit message: Disable collision arm

File: mirte_description/mirte_master_description/urdf/arm.xacro (robot description, xacro)
@@ -31,4 +31,5 @@
             </material>
         </visual>
+        <xacro:if value="$(arg arm_collision)">
         <collision>
             <origin
@@ -40,5 +41,5 @@
             </geometry>
         </collision>
-    </link>
+</xacro:if>    </link>
     <joint
         name="arm_Rot_joint"
@@ -90,4 +91,5 @@
             </material>
         </visual>
+        <xacro:if value="$(arg arm_collision)">
         <collision>
             <origin
@@ -99,5 +101,5 @@
             </geometry>
         </collision>
-    </link>
+</xacro:if>    </link>
     <joint
         name="arm_Shoulder_joint"
@@ -149,4 +151,5 @@
             </material>
         </visual>
+        <xacro:if value="$(arg arm_collision)">
         <collision>
             <origin
@@ -158,5 +161,5 @@
             </geometry>
         </collision>
-    </link>
+</xacro:if>    </link>
     <joint
         name="arm_Elbow_joint"
@@ -208,4 +211,5 @@
             </material>
         </visual>
+        <xacro:if value="$(arg arm_collision)">
         <collision>
             <origin
@@ -217,5 +221,5 @@
             </geometry>
         </collision>
-    </link>
+</xacro:if>    </link>
     <joint
         name="arm_Wrist_joint"
@@ -267,4 +271,5 @@
             </material>
         </visual>
+        <xacro:if value="$(arg arm_collision)">
         <collision>
             <origin
@@ -276,5 +281,5 @@
             </geometry>
         </collision>
-    </link>
+</xacro:if>    </link>
     <joint
         name="Gripper_joint"
@@ -326,4 +331,5 @@
             </material>
         </visual>
+        <xacro:if value="$(arg arm_collision)">
         <collision>
             <origin
@@ -335,5 +341,5 @@
             </geometry>
         </collision>
-    </link>
+</xacro:if>    </link>
     <joint
         name="_gripper_link_joint_r"
@@ -385,4 +391,5 @@
             </material>
         </visual>
+        <xacro:if value="$(arg arm_collision)">
         <collision>
             <origin
@@ -394,5 +401,5 @@
             </geometry>
         </collision>
-    </link>
+</xacro:if>    </link>
     <joint
         name="gripper_finger_joint_r"
@@ -443,4 +450,5 @@
             </material>
         </visual>
+        <xacro:if value="$(arg arm_collision)">
         <collision>
             <origin
@@ -452,5 +460,5 @@
             </geometry>
         </collision>
-    </link>
+</xacro:if>    </link>
     <joint
         name="_gripper_link_joint_l"
@@ -502,4 +510,5 @@
             </material>
         </visual>
+        <xacro:if value="$(arg arm_collision)">
         <collision>
             <origin
@@ -511,5 +520,5 @@
             </geometry>
         </collision>
-    </link>
+</xacro:if>    </link>
     <joint
         name="gripper_finger_joint_l"
@@ -560,4 +569,5 @@
             </material>
         </visual>
+        <xacro:if value="$(arg arm_collision)">
         <collision>
             <origin
@@ -569,5 +579,5 @@
             </geometry>
         </collision>
-    </link>
+</xacro:if>    </link>
     <joint
         name="_Gripper_joint_r"

File: mirte_description/mirte_master_description/urdf/mirte_master.xacro (robot description, xacro)
@@ -8,6 +8,7 @@
   <xacro:arg name="sonar_enable" default="True" />
   <xacro:arg name="lidar_enable" default="True" />
-  <xacro:arg name="depth_camera_enable" default="True" />
-  <xacro:arg name="imu_enable" default="True" />
+  <xacro:arg name="depth_camera_enable" default="False" />
+  <xacro:arg name="imu_enable" default="False" />
+  <xacro:arg name="arm_collision" default="False" />
   <xacro:property name="camera_name" value="camera" lazy_eval="False"/>
   <xacro:property name="namespace" value="" scope="global" lazy_eval="False"/>

Commit message: add collide_bitmask

File: mirte_description/mirte_master_description/urdf/arm.xacro (robot description, xacro)
@@ -40,4 +40,9 @@
                     filename="file://$(find mirte_master_description)/meshes/arm_Rot.STL" />
             </geometry>
+            <surface>
+                <contact>
+                    <collide_bitmask>0x01</collide_bitmask>
+                </contact>
+            </surface>
         </collision>
 </xacro:if>    </link>
@@ -100,4 +105,9 @@
                     filename="file://$(find mirte_master_description)/meshes/arm_Shoulder.STL" />
             </geometry>
+            <surface>
+                <contact>
+                    <collide_bitmask>0x01</collide_bitmask>
+                </contact>
+            </surface>
         </collision>
 </xacro:if>    </link>
@@ -160,4 +170,9 @@
                     filename="file://$(find mirte_master_description)/meshes/arm_Elbow.STL" />
             </geometry>
+            <surface>
+                <contact>
+                    <collide_bitmask>0x01</collide_bitmask>
+                </contact>
+            </surface>
         </collision>
 </xacro:if>    </link>
@@ -220,4 +235,9 @@
                     filename="file://$(find mirte_master_description)/meshes/arm_Wrist.STL" />
             </geometry>
+            <surface>
+                <contact>
+                    <collide_bitmask>0x01</collide_bitmask>
+                </contact>
+            </surface>
         </collision>
 </xacro:if>    </link>
@@ -280,4 +300,9 @@
                     filename="file://$(find mirte_master_description)/meshes/Gripper.STL" />
             </geometry>
+            <surface>
+                <contact>
+                    <collide_bitmask>0x01</collide_bitmask>
+                </contact>
+            </surface>
         </collision>
 </xacro:if>    </link>
@@ -340,4 +365,9 @@
                     filename="file://$(find mirte_master_description)/meshes/_gripper_link_r.STL" />
             </geometry>
+            <surface>
+                <contact>
+                    <collide_bitmask>0x01</collide_bitmask>
+                </contact>
+            </surface>
         </collision>
 </xacro:if>    </link>
@@ -400,4 +430,9 @@
                     filename="file://$(find mirte_master_description)/meshes/gripper_finger_r.STL" />
             </geometry>
+            <surface>
+                <contact>
+                    <collide_bitmask>0x01</collide_bitmask>
+                </contact>
+            </surface>
         </collision>
 </xacro:if>    </link>
@@ -459,4 +494,9 @@
                     filename="file://$(find mirte_master_description)/meshes/_gripper_link_l.STL" />
             </geometry>
+            <surface>
+                <contact>
+                    <collide_bitmask>0x01</collide_bitmask>
+                </contact>
+            </surface>
         </collision>
 </xacro:if>    </link>
@@ -519,4 +559,9 @@
                     filename="file://$(find mirte_master_description)/meshes/gripper_finger_l.STL" />
             </geometry>
+            <surface>
+                <contact>
+                    <collide_bitmask>0x01</collide_bitmask>
+                </contact>
+            </surface>
         </collision>
 </xacro:if>    </link>
@@ -578,4 +623,9 @@
                     filename="file://$(find mirte_master_description)/meshes/_Gripper_r.STL" />
             </geometry>
+            <surface>
+                <contact>
+                    <collide_bitmask>0x01</collide_bitmask>
+                </contact>
+            </surface>
         </collision>
 </xacro:if>    </link>

File: mirte_description/mirte_master_description/urdf/flag.xacro (robot description, xacro)
@@ -33,4 +33,9 @@
             filename="package://mirte_master_description/meshes/flag.STL" />
         </geometry>
+        <surface>
+            <contact>
+                <collide_bitmask>0x01</collide_bitmask>
+            </contact>
+        </surface>
       </collision>
     </link>

File: mirte_description/mirte_master_description/urdf/lidar.xacro (robot description, xacro)
@@ -38,4 +38,9 @@
           filename="file://$(find mirte_master_description)/meshes/lidar.STL" />
       </geometry>
+      <surface>
+        <contact>
+            <collide_bitmask>0x01</collide_bitmask>
+        </contact>
+      </surface>
     </collision>
   </link>

File: mirte_description/mirte_master_description/urdf/mirte_master.xacro (robot description, xacro)
@@ -33,5 +33,13 @@
   </xacro:if>
   <xacro:if value="$(arg imu_enable)">
-    <link name="imu_link" />
+    <link name="imu_link">
+      <collision>
+        <surface>
+              <contact>
+              <collide_bitmask>0x01</collide_bitmask>
+              </contact>
+        </surface>
+      </collision>
+    </link>
     <joint name="imu_joint" type="fixed">
       <origin xyz="0 0 0.10" />
@@ -40,5 +48,13 @@
     </joint>
   </xacro:if>
-  <link name="base_link" />
+  <link name="base_link">
+    <collision>
+      <surface>
+            <contact>
+            <collide_bitmask>0x01</collide_bitmask>
+            </contact>
+      </surface>
+    </collision>
+  </link>
   <gazebo reference="base_link">
      <kinematic>1</kinematic>
@@ -74,4 +90,9 @@
         <box size="0.19 0.28 0.06" />
       </geometry>
+      <surface>
+        <contact>
+          <collide_bitmask>0x01</collide_bitmask>
+        </contact>
+      </surface>
     </collision>
     <collision>
@@ -80,4 +101,9 @@
         <box size="0.18 0.16 0.05" />
       </geometry>
+      <surface>
+        <contact>
+          <collide_bitmask>0x01</collide_bitmask>
+        </contact>
+      </surface>
     </collision>
     <collision>
@@ -86,4 +112,9 @@
         <box size="0.013 0.03 0.025" />
       </geometry>
+      <surface>
+        <contact>
+          <collide_bitmask>0x01</collide_bitmask>
+        </contact>
+      </surface>
     </collision>
     <collision>
@@ -92,4 +123,9 @@
         <box size="0.013 0.04 0.025" />
       </geometry>
+      <surface>
+        <contact>
+          <collide_bitmask>0x01</collide_bitmask>
+        </contact>
+      </surface>
     </collision>
   </link>
@@ -150,4 +186,11 @@
         </material>
       </visual>
+      <collision>
+        <surface>
+            <contact>
+            <collide_bitmask>0x01</collide_bitmask>
+            </contact>
+        </surface>
+      </collision>
     </link>
     <joint
@@ -163,5 +206,13 @@
   </xacro:if>
   <xacro:property name="wheel_zoff" value="0.05"/>
-  <link name="base_footprint"/>
+  <link name="base_footprint">
+    <collision>
+      <surface>
+            <contact>
+            <collide_bitmask>0x01</collide_bitmask>
+            </contact>
+      </surface>
+    </collision>
+  </link>
   <joint name="base_joint" type="fixed">
     <parent link="base_link"/>
@@ -175,5 +226,13 @@
       <child link="link_chassis" />
     </joint>
-    <link name="link_chassis" />
+    <link name="link_chassis">
+    <collision>
+      <surface>
+            <contact>
+            <collide_bitmask>0x01</collide_bitmask>
+            </contact>
+      </surface>
+    </collision>
+    </link>
     <xacro:ultrasonic_sensor name="left_front">
       <origin
@@ -239,4 +298,9 @@
             filename="file://$(find mirte_master_description)/meshes/screen.STL" />
         </geometry>
+        <surface>
+          <contact>
+            <collide_bitmask>0x01</collide_bitmask>
+          </contact>
+        </surface>
       </collision>
     </link>

File: mirte_description/mirte_master_description/urdf/mirte_master_base.gazebo.xacro (robot description, xacro)
@@ -21,4 +21,11 @@
       <pose>0 0 0 0 0 0</pose>
     </sensor>
+    <collision>
+      <surface>
+          <contact>
+          <collide_bitmask>0x01</collide_bitmask>
+          </contact>
+      </surface>
+    </collision>
    </gazebo>
   </xacro:if>
@@ -26,4 +33,11 @@
     <material>Gazebo/White</material>
     <gravity>true</gravity>
+    <collision>
+      <surface>
+          <contact>
+          <collide_bitmask>0x01</collide_bitmask>
+          </contact>
+      </surface>
+    </collision>
   </gazebo>
   <xacro:include filename="$(find mirte_master_description)/urdf/wheel.gazebo.xacro" />

File: mirte_description/mirte_master_description/urdf/orbbec_astra_plus_pro.xacro (robot description, xacro)
@@ -25,4 +25,11 @@
                     <inertia ixx="0.0001" ixy="0.0" ixz="0.0" iyy="0.0001" iyz="0.0" izz="0.0001" />
                </inertial>
+               <collision>
+                    <surface>
+                         <contact>
+                         <collide_bitmask>0x01</collide_bitmask>
+                         </contact>
+                    </surface>
+               </collision>
           </link>
           <joint name="${name}_rgb_optical_joint" type="fixed">
@@ -37,4 +44,11 @@
                     <inertia ixx="0.0001" ixy="0.0" ixz="0.0" iyy="0.0001" iyz="0.0" izz="0.0001" />
                </inertial-->
+               <collision>
+                    <surface>
+                         <contact>
+                         <collide_bitmask>0x01</collide_bitmask>
+                         </contact>
+                    </surface>
+               </collision>
           </link>
           <joint name="${name}_joint" type="fixed">
@@ -59,4 +73,9 @@
                          <box size="0.0370 .1650 0.0350" />
                     </geometry>
+                    <surface>
+                         <contact>
+                              <collide_bitmask>0x01</collide_bitmask>
+                         </contact>
+                    </surface>
                </collision>
                <inertial>
@@ -80,4 +99,11 @@
                     <inertia ixx="0.001" ixy="0.0" ixz="0.0" iyy="0.001" iyz="0.0" izz="0.001" />
                </inertial-->
+               <collision>
+                    <surface>
+                         <contact>
+                         <collide_bitmask>0x01</collide_bitmask>
+                         </contact>
+                    </surface>
+               </collision>
           </link>
           <joint name="${name}_depth_optical_joint" type="fixed">
@@ -92,4 +118,11 @@
                     <inertia ixx="0.0001" ixy="0.0" ixz="0.0" iyy="0.0001" iyz="0.0" izz="0.0001" />
                </inertial-->
+               <collision>
+                    <surface>
+                         <contact>
+                         <collide_bitmask>0x01</collide_bitmask>
+                         </contact>
+                    </surface>
+               </collision>
           </link>
           <!-- RGBD sensor for simulation, same as Kinect -->

File: mirte_description/mirte_master_description/urdf/ultrasonic.xacro (robot description, xacro)
@@ -19,4 +19,11 @@
         <material name="blue" />
       </visual>
+      <collision>
+        <surface>
+            <contact>
+            <collide_bitmask>0x01</collide_bitmask>
+            </contact>
+        </surface>
+      </collision>
     </link>
     <gazebo reference="base_sonar_${name}">

File: mirte_description/mirte_master_description/urdf/wheel.gazebo.xacro (robot description, xacro)
@@ -8,4 +8,11 @@
             <mu2>0.0</mu2>
             <material>Gazebo/DarkGrey</material>
+            <collision>
+                <surface>
+                    <contact>
+                    <collide_bitmask>0x01</collide_bitmask>
+                    </contact>
+                </surface>
+            </collision>
         </gazebo>
     </xacro:macro>

File: mirte_description/mirte_master_description/urdf/wheel.xacro (robot description, xacro)
@@ -29,4 +29,9 @@
         <cylinder radius="${wheel_radius}" length="${wheel_length}" />
       </geometry>
+      <surface>
+        <contact>
+          <collide_bitmask>0x01</collide_bitmask>
+        </contact>
+      </surface>
     </collision>
   </link>
